File: Charge-Seed-Breakout/KiCad/Charge-Seed-Breakout.kicad_pcb (KiCad board)
At the start: 2 copper layers, 175 x 101 mm, 10 parts, among them J1 Screw_01x10, J10 Screw_01x10, J2 Screw_01x10, J3 Pin, J4 Socket, J5 Socket, J6 Socket, J7 Socket, J8 Pin, J9 Screw_01x10

Commit message: 1st Render Updates
Parts:
- moved J1 7.62 mm to (124.5, 86.4)
- moved J2 7.62 mm to (124.5, 113.4)
- moved J3 7.62 mm to (132.1, 86.4)
- moved J4 7.62 mm to (139.7, 86.4)
- moved J5 7.62 mm to (152.4, 86.4)
- moved J6 7.62 mm to (167.6, 86.4)
- moved J7 7.62 mm to (180.3, 86.4)
- moved J8 7.62 mm to (188.0, 86.4)
- moved J9 7.62 mm to (195.6, 109.2)
- moved J10 7.62 mm to (195.6, 136.1)
