File: Charge-Seed-Breakout/KiCad/Charge-Seed-Breakout.kicad_sch (KiCad schematic)
At the start: 10 parts, among them J1 Screw_01x10, J10 Screw_01x10, J2 Screw_01x10, J3 Pin, J4 Socket, J5 Socket, J6 Socket, J7 Socket, J8 Pin, J9 Screw_01x10

Commit message: 1st Render Updates
Other:
- title: Charge-BoB-Seed -> Charge-Seed-Breakout
Changed lines of the file:
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@@
 	(paper "A4")
 	(title_block
-		(title "Charge-BoB-Seed")
+		(title "Charge-Seed-Breakout")
 		(date "2025-09-03")
 		(rev "0.1")
